Commit message: Richer arena (walls + obstacles for SLAM), better robot model, map-frame RViz
World
- gen_track_world.py: add an enclosing arena around the oval - perimeter walls
  plus infield island, corner crates, pillars, drums and cone rows lining the
  straights. All placed >=1 m clear of the racing line (verified), so pure
  pursuit still laps cleanly while the lidar has distinct features to map and
  navigate around. Regenerates ids_world.sdf and oval_track.sdf (24 obstacles).

Robot
- ids_robot.urdf.xacro: layered visuals - upper deck, red front bumper and
  rear antenna, wheel hubs, a lidar mount post and scan ring. Physics
  parameters (wheel radius/separation, inertias, raised casters) unchanged, so
  the detector kinematics are identical.

RViz / match
- gazebo.launch.py: bridge /joint_states so robot_state_publisher completes the
  TF tree and the model renders with turning wheels.
- ids.rviz: enable the laser scan (obstacles now show as scan points, matching
  Gazebo) and add a Map display and the 2D Pose Estimate / 2D Nav Goal tools.

SLAM
- slam.launch.py + config/slam_toolbox.yaml + rviz/slam.rviz: online-async
  mapping. The robot laps the oval under pure pursuit and maps the arena with
  no teleop; map frame view with Nav goal tools. `ids slam` runs it.
- setup.py installs config/; package.xml declares slam_toolbox.

Co-Authored-By: Claude Opus 5.5 <noreply@anthropic.com>
Claude-Session: https://claude.ai/code/session_01XAf5D3tTXwvzgMJCgLAVVU

File: src/physguard/urdf/ids_robot.urdf.xacro (robot description, xacro)
@@ -42,7 +42,10 @@
   <!-- ======== materials ======== -->
   <material name="chassis_blue"><color rgba="0.08 0.31 0.61 1"/></material>
+  <material name="deck_slate"><color rgba="0.20 0.24 0.30 1"/></material>
   <material name="marker_white"><color rgba="0.95 0.95 0.95 1"/></material>
-  <material name="wheel_black"><color rgba="0.12 0.12 0.12 1"/></material>
+  <material name="wheel_black"><color rgba="0.10 0.10 0.10 1"/></material>
+  <material name="hub_grey"><color rgba="0.62 0.65 0.69 1"/></material>
   <material name="lidar_dark"><color rgba="0.10 0.10 0.10 1"/></material>
+  <material name="accent_red"><color rgba="0.82 0.20 0.18 1"/></material>
   <!-- ======== macros ======== -->
   <xacro:macro name="box_inertia" params="m x y z">
@@ -59,4 +62,9 @@
         <geometry><cylinder radius="${wheel_radius}" length="${wheel_width}"/></geometry>
         <material name="wheel_black"/>
+      </visual>
+      <visual name="hub">
+        <origin xyz="0 0 0" rpy="1.5707963 0 0"/>
+        <geometry><cylinder radius="${wheel_radius*0.5}" length="${wheel_width*1.08}"/></geometry>
+        <material name="hub_grey"/>
       </visual>
       <collision>
@@ -109,8 +117,23 @@
       <material name="chassis_blue"/>
     </visual>
+    <visual name="deck">
+      <origin xyz="-0.01 0 ${chassis_z + 0.02}" rpy="0 0 0"/>
+      <geometry><box size="0.22 0.18 0.04"/></geometry>
+      <material name="deck_slate"/>
+    </visual>
+    <visual name="front_bumper">
+      <origin xyz="${chassis_x/2.0} 0 ${chassis_z/2.0 - 0.005}" rpy="0 0 0"/>
+      <geometry><box size="0.02 0.22 0.05"/></geometry>
+      <material name="accent_red"/>
+    </visual>
     <visual name="front_marker">
       <origin xyz="${chassis_x/2.0 - 0.02} 0 ${chassis_z/2.0 + 0.035}" rpy="0 0 0"/>
       <geometry><box size="0.04 0.18 0.01"/></geometry>
       <material name="marker_white"/>
+    </visual>
+    <visual name="antenna">
+      <origin xyz="${-chassis_x/2.0 + 0.03} 0.07 ${chassis_z + 0.08}" rpy="0 0 0"/>
+      <geometry><cylinder radius="0.004" length="0.16"/></geometry>
+      <material name="accent_red"/>
     </visual>
     <collision>
@@ -126,7 +149,17 @@
   <!-- ======== lidar ======== -->
   <link name="lidar_link">
-    <visual>
+    <visual name="mount">
+      <origin xyz="0 0 -0.035" rpy="0 0 0"/>
+      <geometry><cylinder radius="0.015" length="0.05"/></geometry>
+      <material name="deck_slate"/>
+    </visual>
+    <visual name="drum">
       <geometry><cylinder radius="0.04" length="0.04"/></geometry>
       <material name="lidar_dark"/>
+    </visual>
+    <visual name="scan_ring">
+      <origin xyz="0 0 0.012" rpy="0 0 0"/>
+      <geometry><cylinder radius="0.041" length="0.008"/></geometry>
+      <material name="accent_red"/>
     </visual>
     <collision>
