Commit message: Rebuild the Gazebo layer so RViz and Gazebo always agree
- Robot rests on three contacts (two wheels + one rear caster) with sphere
  wheel collisions, so the drive wheels keep traction and wheel odometry
  stays within millimetres of the true pose (was drifting ~3.8 m)
- Gazebo OdometryPublisher adds /ground_truth; new sim_frames node publishes
  odom->base_link from /odom and world->odom from ground truth
- Single bridge config (config/gz_bridge.yaml), no /tf bridge
- Controller and IDS start on spawn completion, not a timer
- New world-frame RViz layout; track_viz frame is a parameter
- Detector still runs on raw wheel /odom; pose_topic selects what the
  controller and scorer use (default /ground_truth)

File: src/physguard/urdf/ids_robot.urdf.xacro (robot description, xacro)
@@ -8,47 +8,64 @@
 ================================================================================
  Description
- Differential-drive robot description for the IDS bench, matching the
- articubot_one platform the detector targets:
-     wheel radius 32.5 mm, wheel separation 250 mm, two casters, RPLIDAR A2M8.
- Structure
-   base_link (chassis, root)
-     +- left_wheel_joint  (continuous)  -> left_wheel
-     +- right_wheel_joint (continuous)  -> right_wheel
-     +- front_caster_joint (fixed)      -> front_caster   (frictionless)
-     +- rear_caster_joint  (fixed)      -> rear_caster    (frictionless)
-     +- lidar_joint        (fixed)      -> lidar_link     (gpu_lidar sensor)
- The gz-sim DiffDrive system drives the wheel joints, consumes /cmd_vel and
- publishes /odom and the odom->base_link TF. robot_state_publisher publishes
- the fixed base_link->{wheels,casters,lidar} transforms from this file, so the
- same description serves Gazebo, RViz2 and (later) the real robot.
- Casters sit 3 mm clear of the ground so the drive wheels carry the load;
- coplanar contacts let the frictionless casters steal traction and the wheels
- slip, which corrupts odometry.
+ Differential-drive robot for the Gazebo Harmonic bench, built to match the
+ real articubot_one: wheel radius 32.5 mm, wheel separation 250 mm, one rear
+ caster, RPLIDAR on top. Every geometric number lives in ONE place (the
+ properties below) and is reused by the links, the DiffDrive system and the
+ detector's assumptions, so the sim cannot drift out of agreement with itself.
+ Structure (base_link is at the wheel axle, centred between the wheels)
+   base_link            chassis, deck, bumper
+     +- left_wheel_joint  (continuous) -> left_wheel
+     +- right_wheel_joint (continuous) -> right_wheel
+     +- caster_joint      (fixed)      -> caster        rear, near-frictionless
+     +- lidar_joint       (fixed)      -> lidar_link    gpu_lidar -> /scan
+ Contact design (why this robot does not drift)
+   * Three ground contacts: two drive wheels + one rear caster. Three points
+     are statically determinate, so the load split is fixed by geometry and
+     the drive wheels can never be unloaded. (Four rigid contacts - the old
+     model - let the physics engine split the load arbitrarily, the wheels
+     lost normal force and slipped, and wheel odometry ran ahead.)
+   * The chassis centre of mass sits between the axle and the caster, so the
+     wheels carry about 2/3 of the weight and keep traction.
+   * Wheel collisions are spheres of the wheel radius: one contact point
+     directly under each hub, so the effective radius and track width in the
+     physics engine are exactly wheel_radius and wheel_sep.
+ Gazebo systems
+   DiffDrive           /cmd_vel in, wheel odometry out on /odom (its TF goes
+                       to an unbridged gz topic; sim_frames publishes the TF)
+   JointStatePublisher /joint_states, for robot_state_publisher
+   OdometryPublisher   GROUND TRUTH pose of base_link in 'world' on
+                       /ground_truth. Used for the world->odom correction so
+                       RViz mirrors Gazebo, by the controller, and for metrics.
+                       The detector never sees it; it uses wheel /odom.
 ================================================================================
 -->
 <robot name="ids_robot" xmlns:xacro="http://www.ros.org/wiki/xacro">
-  <!-- ======== parameters ======== -->
-  <xacro:property name="wheel_radius"    value="0.0325"/>
-  <xacro:property name="wheel_width"     value="0.020"/>
-  <xacro:property name="wheel_sep"       value="0.250"/>
-  <xacro:property name="chassis_x"       value="0.30"/>
-  <xacro:property name="chassis_y"       value="0.22"/>
-  <xacro:property name="chassis_z"       value="0.08"/>
-  <xacro:property name="chassis_mass"    value="1.5"/>
-  <xacro:property name="wheel_mass"      value="0.10"/>
-  <xacro:property name="caster_radius"   value="0.020"/>
-  <!-- caster centre height: sphere bottom 3 mm above ground -->
-  <xacro:property name="caster_z"        value="${-wheel_radius + caster_radius + 0.003}"/>
+  <!-- ======== geometry: the single source of truth ======== -->
+  <xacro:property name="wheel_radius"   value="0.0325"/>
+  <xacro:property name="wheel_width"    value="0.026"/>
+  <xacro:property name="wheel_sep"      value="0.250"/>
+  <xacro:property name="wheel_mass"     value="0.10"/>
+  <xacro:property name="chassis_x"      value="0.30"/>
+  <xacro:property name="chassis_y"      value="0.20"/>
+  <xacro:property name="chassis_z"      value="0.08"/>
+  <xacro:property name="chassis_mass"   value="1.5"/>
+  <!-- chassis centre is behind the axle, towards the caster -->
+  <xacro:property name="chassis_cx"     value="-0.06"/>
+  <xacro:property name="caster_radius"  value="0.020"/>
+  <xacro:property name="caster_x"       value="-0.17"/>
+  <!-- caster bottom exactly at ground level (ground is z = -wheel_radius) -->
+  <xacro:property name="caster_z"       value="${-wheel_radius + caster_radius}"/>
+  <!-- lidar scan plane sits above every other visual (gpu_lidar sees visuals) -->
+  <xacro:property name="lidar_z"        value="${chassis_z + 0.05}"/>
   <!-- ======== materials ======== -->
   <material name="chassis_blue"><color rgba="0.08 0.31 0.61 1"/></material>
   <material name="deck_slate"><color rgba="0.20 0.24 0.30 1"/></material>
-  <material name="marker_white"><color rgba="0.95 0.95 0.95 1"/></material>
   <material name="wheel_black"><color rgba="0.10 0.10 0.10 1"/></material>
   <material name="hub_grey"><color rgba="0.62 0.65 0.69 1"/></material>
-  <material name="lidar_dark"><color rgba="0.10 0.10 0.10 1"/></material>
   <material name="accent_red"><color rgba="0.82 0.20 0.18 1"/></material>
-  <!-- ======== macros ======== -->
-  <xacro:macro name="box_inertia" params="m x y z">
-    <inertial>
+  <!-- ======== inertia helpers ======== -->
+  <xacro:macro name="box_inertia" params="m x y z ox:=0 oy:=0 oz:=0">
+    <inertial>
+      <origin xyz="${ox} ${oy} ${oz}" rpy="0 0 0"/>
       <mass value="${m}"/>
       <inertia ixx="${m*(y*y+z*z)/12.0}" iyy="${m*(x*x+z*z)/12.0}"
@@ -56,24 +73,54 @@
     </inertial>
   </xacro:macro>
+  <!-- wheel spins about the joint's y axis; cylinder inertia expressed in that frame -->
+  <xacro:macro name="wheel_inertia" params="m r h">
+    <inertial>
+      <mass value="${m}"/>
+      <inertia ixx="${m*(3*r*r+h*h)/12.0}" iyy="${m*r*r/2.0}"
+               izz="${m*(3*r*r+h*h)/12.0}" ixy="0" ixz="0" iyz="0"/>
+    </inertial>
+  </xacro:macro>
+  <!-- ======== chassis (root, at the wheel axle) ======== -->
+  <link name="base_link">
+    <visual name="chassis">
+      <origin xyz="${chassis_cx} 0 ${chassis_z/2.0}" rpy="0 0 0"/>
+      <geometry><box size="${chassis_x} ${chassis_y} ${chassis_z}"/></geometry>
+      <material name="chassis_blue"/>
+    </visual>
+    <visual name="deck">
+      <origin xyz="${chassis_cx} 0 ${chassis_z + 0.008}" rpy="0 0 0"/>
+      <geometry><box size="${chassis_x - 0.06} ${chassis_y - 0.04} 0.016"/></geometry>
+      <material name="deck_slate"/>
+    </visual>
+    <visual name="front_bumper">
+      <origin xyz="${chassis_cx + chassis_x/2.0 + 0.008} 0 ${chassis_z/2.0}" rpy="0 0 0"/>
+      <geometry><box size="0.016 ${chassis_y} 0.04"/></geometry>
+      <material name="accent_red"/>
+    </visual>
+    <collision>
+      <origin xyz="${chassis_cx} 0 ${chassis_z/2.0}" rpy="0 0 0"/>
+      <geometry><box size="${chassis_x} ${chassis_y} ${chassis_z}"/></geometry>
+    </collision>
+    <xacro:box_inertia m="${chassis_mass}" x="${chassis_x}" y="${chassis_y}" z="${chassis_z}"
+                       ox="${chassis_cx}" oz="${chassis_z/2.0}"/>
+  </link>
+  <!-- ======== drive wheels ======== -->
   <xacro:macro name="wheel" params="prefix reflect">
     <link name="${prefix}_wheel">
-      <visual>
-        <origin xyz="0 0 0" rpy="1.5707963 0 0"/>
+      <visual name="tyre">
+        <origin xyz="0 0 0" rpy="${pi/2} 0 0"/>
         <geometry><cylinder radius="${wheel_radius}" length="${wheel_width}"/></geometry>
         <material name="wheel_black"/>
       </visual>
       <visual name="hub">
-        <origin xyz="0 0 0" rpy="1.5707963 0 0"/>
+        <origin xyz="0 0 0" rpy="${pi/2} 0 0"/>
         <geometry><cylinder radius="${wheel_radius*0.5}" length="${wheel_width*1.08}"/></geometry>
         <material name="hub_grey"/>
       </visual>
+      <!-- sphere collision: single contact point under the hub -->
       <collision>
-        <origin xyz="0 0 0" rpy="1.5707963 0 0"/>
-        <geometry><cylinder radius="${wheel_radius}" length="${wheel_width}"/></geometry>
+        <geometry><sphere radius="${wheel_radius}"/></geometry>
       </collision>
-      <inertial>
-        <mass value="${wheel_mass}"/>
-        <inertia ixx="2.97e-5" iyy="2.97e-5" izz="5.28e-5" ixy="0" ixz="0" iyz="0"/>
-      </inertial>
+      <xacro:wheel_inertia m="${wheel_mass}" r="${wheel_radius}" h="${wheel_width}"/>
     </link>
     <joint name="${prefix}_wheel_joint" type="continuous">
@@ -84,89 +131,50 @@
     </joint>
     <gazebo reference="${prefix}_wheel">
-      <mu1>1.0</mu1><mu2>1.0</mu2>
+      <mu1>1.0</mu1>
+      <mu2>1.0</mu2>
     </gazebo>
   </xacro:macro>
-  <xacro:macro name="caster" params="prefix x">
-    <link name="${prefix}_caster">
-      <visual>
-        <geometry><sphere radius="${caster_radius}"/></geometry>
-        <material name="wheel_black"/>
-      </visual>
-      <collision>
-        <geometry><sphere radius="${caster_radius}"/></geometry>
-      </collision>
-      <inertial>
-        <mass value="0.02"/>
-        <inertia ixx="3.2e-6" iyy="3.2e-6" izz="3.2e-6" ixy="0" ixz="0" iyz="0"/>
-      </inertial>
-    </link>
-    <joint name="${prefix}_caster_joint" type="fixed">
-      <parent link="base_link"/>
-      <child link="${prefix}_caster"/>
-      <origin xyz="${x} 0 ${caster_z}" rpy="0 0 0"/>
-    </joint>
-    <gazebo reference="${prefix}_caster">
-      <mu1>0.0</mu1><mu2>0.0</mu2>
-    </gazebo>
-  </xacro:macro>
-  <!-- ======== chassis (root) ======== -->
-  <link name="base_link">
-    <visual>
-      <origin xyz="0 0 ${chassis_z/2.0}" rpy="0 0 0"/>
-      <geometry><box size="${chassis_x} ${chassis_y} ${chassis_z}"/></geometry>
-      <material name="chassis_blue"/>
-    </visual>
-    <visual name="deck">
-      <origin xyz="-0.01 0 ${chassis_z + 0.02}" rpy="0 0 0"/>
-      <geometry><box size="0.22 0.18 0.04"/></geometry>
-      <material name="deck_slate"/>
-    </visual>
-    <visual name="front_bumper">
-      <origin xyz="${chassis_x/2.0} 0 ${chassis_z/2.0 - 0.005}" rpy="0 0 0"/>
-      <geometry><box size="0.02 0.22 0.05"/></geometry>
-      <material name="accent_red"/>
-    </visual>
-    <visual name="front_marker">
-      <origin xyz="${chassis_x/2.0 - 0.02} 0 ${chassis_z/2.0 + 0.035}" rpy="0 0 0"/>
-      <geometry><box size="0.04 0.18 0.01"/></geometry>
-      <material name="marker_white"/>
-    </visual>
-    <visual name="antenna">
-      <origin xyz="${-chassis_x/2.0 + 0.03} 0.07 ${chassis_z + 0.08}" rpy="0 0 0"/>
-      <geometry><cylinder radius="0.004" length="0.16"/></geometry>
-      <material name="accent_red"/>
-    </visual>
-    <collision>
-      <origin xyz="0 0 ${chassis_z/2.0}" rpy="0 0 0"/>
-      <geometry><box size="${chassis_x} ${chassis_y} ${chassis_z}"/></geometry>
-    </collision>
-    <xacro:box_inertia m="${chassis_mass}" x="${chassis_x}" y="${chassis_y}" z="${chassis_z}"/>
-  </link>
   <xacro:wheel prefix="left"  reflect="1"/>
   <xacro:wheel prefix="right" reflect="-1"/>
-  <xacro:caster prefix="front" x="0.11"/>
-  <xacro:caster prefix="rear"  x="-0.11"/>
+  <!-- ======== rear caster (near-frictionless sphere) ======== -->
+  <link name="caster">
+    <visual>
+      <geometry><sphere radius="${caster_radius}"/></geometry>
+      <material name="hub_grey"/>
+    </visual>
+    <collision>
+      <geometry><sphere radius="${caster_radius}"/></geometry>
+    </collision>
+    <inertial>
+      <mass value="0.02"/>
+      <inertia ixx="3.2e-6" iyy="3.2e-6" izz="3.2e-6" ixy="0" ixz="0" iyz="0"/>
+    </inertial>
+  </link>
+  <joint name="caster_joint" type="fixed">
+    <parent link="base_link"/>
+    <child link="caster"/>
+    <origin xyz="${caster_x} 0 ${caster_z}" rpy="0 0 0"/>
+  </joint>
+  <gazebo reference="caster">
+    <mu1>0.001</mu1>
+    <mu2>0.001</mu2>
+  </gazebo>
   <!-- ======== lidar ======== -->
   <link name="lidar_link">
-    <visual name="mount">
-      <origin xyz="0 0 -0.035" rpy="0 0 0"/>
-      <geometry><cylinder radius="0.015" length="0.05"/></geometry>
-      <material name="deck_slate"/>
-    </visual>
     <visual name="drum">
-      <geometry><cylinder radius="0.04" length="0.04"/></geometry>
-      <material name="lidar_dark"/>
+      <geometry><cylinder radius="0.035" length="0.03"/></geometry>
+      <material name="wheel_black"/>
     </visual>
     <visual name="scan_ring">
       <origin xyz="0 0 0.012" rpy="0 0 0"/>
-      <geometry><cylinder radius="0.041" length="0.008"/></geometry>
+      <geometry><cylinder radius="0.036" length="0.006"/></geometry>
       <material name="accent_red"/>
     </visual>
     <collision>
-      <geometry><cylinder radius="0.04" length="0.04"/></geometry>
+      <geometry><cylinder radius="0.035" length="0.03"/></geometry>
     </collision>
     <inertial>
-      <mass value="0.1"/>
-      <inertia ixx="4.5e-5" iyy="4.5e-5" izz="8.0e-5" ixy="0" ixz="0" iyz="0"/>
+      <mass value="0.10"/>
+      <inertia ixx="3.8e-5" iyy="3.8e-5" izz="6.1e-5" ixy="0" ixz="0" iyz="0"/>
     </inertial>
   </link>
@@ -174,7 +182,6 @@
     <parent link="base_link"/>
     <child link="lidar_link"/>
-    <origin xyz="0.02 0 ${chassis_z + 0.03}" rpy="0 0 0"/>
+    <origin xyz="0 0 ${lidar_z}" rpy="0 0 0"/>
   </joint>
-  <!-- ======== Gazebo: lidar sensor ======== -->
   <gazebo reference="lidar_link">
     <sensor name="lidar" type="gpu_lidar">
@@ -187,11 +194,13 @@
           <min_angle>-3.14159</min_angle><max_angle>3.14159</max_angle>
         </horizontal></scan>
-        <range><min>0.12</min><max>12.0</max><resolution>0.01</resolution></range>
+        <range><min>0.15</min><max>12.0</max><resolution>0.01</resolution></range>
       </lidar>
-      <always_on>1</always_on><visualize>true</visualize>
+      <always_on>1</always_on>
+      <visualize>false</visualize>
     </sensor>
   </gazebo>
-  <!-- ======== Gazebo: differential drive + joint states ======== -->
+  <!-- ======== Gazebo systems ======== -->
   <gazebo>
+    <!-- wheel odometry: what the real robot will have, and what the IDS uses -->
     <plugin filename="gz-sim-diff-drive-system" name="gz::sim::systems::DiffDrive">
       <left_joint>left_wheel_joint</left_joint>
@@ -202,11 +211,12 @@
       <topic>/cmd_vel</topic>
       <odom_topic>/odom</odom_topic>
-      <tf_topic>/tf</tf_topic>
+      <!-- TF left on a private gz topic; sim_frames publishes odom->base_link -->
+      <tf_topic>/model/ids_robot/tf_wheel_odom</tf_topic>
       <frame_id>odom</frame_id>
       <child_frame_id>base_link</child_frame_id>
-      <max_linear_acceleration>1.6</max_linear_acceleration>
-      <min_linear_acceleration>-1.6</min_linear_acceleration>
-      <max_angular_acceleration>4.0</max_angular_acceleration>
-      <min_angular_acceleration>-4.0</min_angular_acceleration>
+      <max_linear_acceleration>1.0</max_linear_acceleration>
+      <min_linear_acceleration>-1.0</min_linear_acceleration>
+      <max_angular_acceleration>3.0</max_angular_acceleration>
+      <min_angular_acceleration>-3.0</min_angular_acceleration>
     </plugin>
     <plugin filename="gz-sim-joint-state-publisher-system"
@@ -214,4 +224,14 @@
       <topic>/joint_states</topic>
     </plugin>
+    <!-- ground truth: exact pose of base_link in the world -->
+    <plugin filename="gz-sim-odometry-publisher-system"
+            name="gz::sim::systems::OdometryPublisher">
+      <odom_frame>world</odom_frame>
+      <robot_base_frame>base_link</robot_base_frame>
+      <odom_topic>/ground_truth</odom_topic>
+      <tf_topic>/model/ids_robot/tf_ground_truth</tf_topic>
+      <odom_publish_frequency>50</odom_publish_frequency>
+      <dimensions>2</dimensions>
+    </plugin>
   </gazebo>
 </robot>
